Commit message: add urdf

File: tests/fixtures/urdf/simple_robot.urdf (robot description, URDF)
Before this commit: robot test_bot, 2 links, 1 joints
Links:
- link base_link: geometry collision box size=0.4 0.2 0.1; visual mesh filename=package://gobot_test_robot/meshes/base_visual.dae

Commit message: add urdf import

File: tests/fixtures/urdf/simple_robot.urdf (robot description, URDF)
Before this commit: robot test_bot, 2 links, 1 joints
Links:
- link base_link: geometry collision box size=0.4 0.2 0.1; visual mesh filename=package://gobot_test_robot/meshes/base_visual.dae scale=0.1 0.2 0.3
